File: leddy.kicad_pcb (KiCad board)
At the start: 4 copper layers, 86.8 x 60.8 mm, 79 parts, among them J1 hole 1, J2 hole 1, J3 hole 1, J4 hole 1, J5 umbrella support, J6 BARREL_JACK, J7 OPEN HARDWARE, J8 label_power-in, Q1 ZXMP6A13GTA, SW1 SW_DPST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

Commit message: added simple debouncing circuit (to be tested)
Parts:
- added C5: 0.1uF, Capacitors_SMD:C_0603_HandSoldering, F.Cu at (149.4, 105.6)
- added R11: 1M, Resistors_SMD:R_0603_HandSoldering, F.Cu at (145.8, 105.6)
- added R12: 1M, Resistors_SMD:R_0603_HandSoldering, F.Cu at (152.8, 105.6)
Connections:
- SW1 pad 2: Vref -> Net-(SW1-Pad2)
- SW1 pad 3: Net-(SW1-Pad1) -> Net-(C5-Pad1)
- SW1 pad 4: Vref -> Net-(SW1-Pad4)
- U2 pad 14: Net-(SW1-Pad1) -> Net-(C5-Pad1)
Changed lines of the file:
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@@
 (kicad_pcb (version 20170123) (host pcbnew no-vcs-found-01f5a12~58~ubuntu14.04.1)
   (general
-    (links 110)
-    (no_connects 110)
+    (links 112)
+    (no_connects 112)
     (area 72.4025 44.924999 210.927381 109.7425)
     (thickness 1.6)
@@
     (tracks 0)
     (zones 0)
-    (modules 79)
-    (nets 78)
+    (modules 82)
+    (nets 82)
   )
   (page A4)
@@
   (net 76 "Net-(R7-Pad2)")
   (net 77 "Net-(F1-Pad2)")
+  (net 78 "Net-(SW1-Pad4)")
+  (net 79 "Net-(SW1-Pad2)")
+  (net 80 "Net-(C5-Pad1)")
+  (net 81 "Net-(R12-Pad2)")
   (net_class Default "This is the default net class."
     (clearance 0.2)
@@
     (add_net "Net-(C2-Pad1)")
     (add_net "Net-(C3-Pad1)")
+    (add_net "Net-(C5-Pad1)")
     (add_net "Net-(D1-Pad1)")
     (add_net "Net-(D10-Pad2)")
@@
     (add_net "Net-(Q1-Pad3)")
     (add_net "Net-(R1-Pad2)")
+    (add_net "Net-(R12-Pad2)")
     (add_net "Net-(R3-Pad2)")
     (add_net "Net-(R4-Pad1)")
@@
     (add_net "Net-(R9-Pad2)")
     (add_net "Net-(SW1-Pad1)")
+    (add_net "Net-(SW1-Pad2)")
+    (add_net "Net-(SW1-Pad4)")
     (add_net "Net-(U1-Pad13)")
     (add_net "Net-(U1-Pad9)")
@@
     (add_net Vref)
   )
+  (module Capacitors_SMD:C_0603_HandSoldering (layer TOP.Cu)
+    (at 149.4 105.6 270)
+    (descr "Capacitor SMD 0603, hand soldering")
+    (tags "capacitor 0603")
+    (attr smd)
+    (fp_text reference C5 (at 0 -1.25 270) (layer F.SilkS)
+      (effects (font (size 1 1) (thickness 0.15)))
+    )
+    (fp_text value 0.1uF (at 0 1.5 270) (layer F.Fab)
+      (effects (font (size 1 1) (thickness 0.15)))
+    )
+    (fp_text user %R (at 0 -1.25 270) (layer F.Fab)
+      (effects (font (size 1 1) (thickness 0.15)))
+    )
+    (fp_line (start -0.8 0.4) (end -0.8 -0.4) (layer F.Fab) (width 0.1))
+    (fp_line (start 0.8 0.4) (end -0.8 0.4) (layer F.Fab) (width 0.1))
+    (fp_line (start 0.8 -0.4) (end 0.8 0.4) (layer F.Fab) (width 0.1))
+    (fp_line (start -0.8 -0.4) (end 0.8 -0.4) (layer F.Fab) (width 0.1))
+    (fp_line (start -0.35 -0.6) (end 0.35 -0.6) (layer F.SilkS) (width 0.12))
+    (fp_line (start 0.35 0.6) (end -0.35 0.6) (layer F.SilkS) (width 0.12))
+    (fp_line (start -1.8 -0.65) (end 1.8 -0.65) (layer F.CrtYd) (width 0.05))
+    (fp_line (start -1.8 -0.65) (end -1.8 0.65) (layer F.CrtYd) (width 0.05))
+    (fp_line (start 1.8 0.65) (end 1.8 -0.65) (layer F.CrtYd) (width 0.05))
+    (fp_line (start 1.8 0.65) (end -1.8 0.65) (layer F.CrtYd) (width 0.05))
+    (pad 1 smd rect (at -0.95 0 270) (size 1.2 0.75) (layers TOP.Cu F.Paste F.Mask)
+      (net 80 "Net-(C5-Pad1)"))
+    (pad 2 smd rect (at 0.95 0 270) (size 1.2 0.75) (layers TOP.Cu F.Paste F.Mask)
+      (net 9 GND))
+    (model Capacitors_SMD.3dshapes/C_0603.wrl
+      (at (xyz 0 0 0))
+      (scale (xyz 1 1 1))
+      (rotate (xyz 0 0 0))
+    )
+  )
+  (module Resistors_SMD:R_0603_HandSoldering (layer TOP.Cu)
+    (at 152.8 105.6 270)
+    (descr "Resistor SMD 0603, hand soldering")
+    (tags "resistor 0603")
+    (attr smd)
+    (fp_text reference R12 (at 0 -1.45 270) (layer F.SilkS)
+      (effects (font (size 1 1) (thickness 0.15)))
+    )
+    (fp_text value 1M (at 0 1.55 270) (layer F.Fab)
+      (effects (font (size 1 1) (thickness 0.15)))
+    )
+    (fp_line (start 1.95 0.7) (end -1.96 0.7) (layer F.CrtYd) (width 0.05))
+    (fp_line (start 1.95 0.7) (end 1.95 -0.7) (layer F.CrtYd) (width 0.05))
+    (fp_line (start -1.96 -0.7) (end -1.96 0.7) (layer F.CrtYd) (width 0.05))
+    (fp_line (start -1.96 -0.7) (end 1.95 -0.7) (layer F.CrtYd) (width 0.05))
+    (fp_line (start -0.5 -0.68) (end 0.5 -0.68) (layer F.SilkS) (width 0.12))
+    (fp_line (start 0.5 0.68) (end -0.5 0.68) (layer F.SilkS) (width 0.12))
+    (fp_line (start -0.8 -0.4) (end 0.8 -0.4) (layer F.Fab) (width 0.1))
+    (fp_line (start 0.8 -0.4) (end 0.8 0.4) (layer F.Fab) (width 0.1))
+    (fp_line (start 0.8 0.4) (end -0.8 0.4) (layer F.Fab) (width 0.1))
+    (fp_line (start -0.8 0.4) (end -0.8 -0.4) (layer F.Fab) (width 0.1))
+    (fp_text user %R (at 0 -1.45 270) (layer F.Fab)
+      (effects (font (size 1 1) (thickness 0.15)))
+    )
+    (pad 2 smd rect (at 1.1 0 270) (size 1.2 0.9) (layers TOP.Cu F.Paste F.Mask)
+      (net 81 "Net-(R12-Pad2)"))
+    (pad 1 smd rect (at -1.1 0 270) (size 1.2 0.9) (layers TOP.Cu F.Paste F.Mask)
+      (net 64 Vref))
+    (model Resistors_SMD.3dshapes/R_0603.wrl
+      (at (xyz 0 0 0))
+      (scale (xyz 1 1 1))
+      (rotate (xyz 0 0 0))
+    )
+  )
+  (module Resistors_SMD:R_0603_HandSoldering (layer TOP.Cu)
+    (at 145.8 105.6 90)
+    (descr "Resistor SMD 0603, hand soldering")
+    (tags "resistor 0603")
+    (attr smd)
+    (fp_text reference R11 (at 0 -1.45 90) (layer F.SilkS)
+      (effects (font (size 1 1) (thickness 0.15)))
+    )
+    (fp_text value 1M (at 0 1.55 90) (layer F.Fab)
+      (effects (font (size 1 1) (thickness 0.15)))
+    )
+    (fp_text user %R (at 0 -1.45 90) (layer F.Fab)
+      (effects (font (size 1 1) (thickness 0.15)))
+    )
+    (fp_line (start -0.8 0.4) (end -0.8 -0.4) (layer F.Fab) (width 0.1))
+    (fp_line (start 0.8 0.4) (end -0.8 0.4) (layer F.Fab) (width 0.1))
+    (fp_line (start 0.8 -0.4) (end 0.8 0.4) (layer F.Fab) (width 0.1))
+    (fp_line (start -0.8 -0.4) (end 0.8 -0.4) (layer F.Fab) (width 0.1))
+    (fp_line (start 0.5 0.68) (end -0.5 0.68) (layer F.SilkS) (width 0.12))
+    (fp_line (start -0.5 -0.68) (end 0.5 -0.68) (layer F.SilkS) (width 0.12))
+    (fp_line (start -1.96 -0.7) (end 1.95 -0.7) (layer F.CrtYd) (width 0.05))
+    (fp_line (start -1.96 -0.7) (end -1.96 0.7) (layer F.CrtYd) (width 0.05))
+    (fp_line (start 1.95 0.7) (end 1.95 -0.7) (layer F.CrtYd) (width 0.05))
+    (fp_line (start 1.95 0.7) (end -1.96 0.7) (layer F.CrtYd) (width 0.05))
+    (pad 1 smd rect (at -1.1 0 90) (size 1.2 0.9) (layers TOP.Cu F.Paste F.Mask)
+      (net 9 GND))
+    (pad 2 smd rect (at 1.1 0 90) (size 1.2 0.9) (layers TOP.Cu F.Paste F.Mask)
+      (net 80 "Net-(C5-Pad1)"))
+    (model Resistors_SMD.3dshapes/R_0603.wrl
+      (at (xyz 0 0 0))
+      (scale (xyz 1 1 1))
+      (rotate (xyz 0 0 0))
+    )
+  )
   (module lib:sw_push4p (layer TOP.Cu)
     (at 137 99.8 270)
@@
       (net 72 "Net-(SW1-Pad1)"))
     (pad 4 smd rect (at 5.5 3 270) (size 3 2) (layers TOP.Cu F.Paste F.Mask)
-      (net 64 Vref))
+      (net 78 "Net-(SW1-Pad4)"))
     (pad 2 smd rect (at -4.572 3 270) (size 3 2) (layers TOP.Cu F.Paste F.Mask)
-      (net 64 Vref))
+      (net 79 "Net-(SW1-Pad2)"))
     (pad 3 smd rect (at 5.5 -4.572 270) (size 3 2) (layers TOP.Cu F.Paste F.Mask)
-      (net 72 "Net-(SW1-Pad1)"))
+      (net 80 "Net-(C5-Pad1)"))
     (model R_discret/switch_push4pinos.wrl
       (at (xyz 0 0 0))
@@
       (net 9 GND))
     (pad 14 smd rect (at 2.95 -0.975 180) (size 1.5 0.45) (layers TOP.Cu F.Paste F.Mask)
-      (net 72 "Net-(SW1-Pad1)"))
+      (net 80 "Net-(C5-Pad1)"))
     (pad 15 smd rect (at 2.95 -1.625 180) (size 1.5 0.45) (layers TOP.Cu F.Paste F.Mask)
       (net 69 "Net-(U2-Pad10)"))

Commit message: started PCB layouting
Parts:
- J5: footprint Mounting_Holes:MountingHole_6.5mm -> Mounting_Holes:MountingHole_8.4mm_M8
- J8: footprint Symbols:Polarity_Center_Positive_6mm_SilkScreen -> lib:Polarity_Center_Positive_3mm_SilkScreen
- SW1: value SW_DPST -> PTS645SM70SMTR92
- moved J7 37.3 mm to (207.0, 96.5)
- moved J1 4.80 mm to (132.4, 51.2)
- moved J2 4.80 mm to (132.4, 104.8)
- moved J8 4.49 mm to (156.0, 56.0)
- moved J6 4.42 mm to (148.4, 61.7)
- moved SW1 1.22 mm to (138.0, 100.5)
- moved F1 1.06 mm to (133.0, 61.5), turned to 90 degrees
- moved C5 0.50 mm to (149.9, 105.6)
- moved R10 0.50 mm to (152.1, 94.2)
- moved R11 0.50 mm to (146.3, 105.6)
- moved R12 0.50 mm to (153.3, 105.6)
- moved R3 0.50 mm to (156.9, 99.6)
- moved R5 0.50 mm to (156.9, 101.2)
- moved R7 0.50 mm to (156.9, 98.0)
- moved R9 0.50 mm to (156.9, 94.4)
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Connections:
- SW1 pad 1: Net-(SW1-Pad1) -> Net-(C5-Pad1)
- SW1 pad 3: Net-(C5-Pad1) -> Net-(SW1-Pad3)
- SW1 pad 4: Net-(SW1-Pad4) -> Net-(R12-Pad2)
- U2 pad 14: Net-(C5-Pad1) -> Net-(U2-Pad14)
Routing:
- added copper zone on F.Cu, net GND
Other:
- board size 86.8 x 60.8 mm -> 83 x 61 mm
- board text added: "VIN: 5-28V"

Commit message: added led current level indication
Parts:
- removed J8: label_power-in, lib:Polarity_Center_Positive_3mm_SilkScreen
- added D51: 29.9V, Diodes_SMD:D_0603, F.Cu at (106.1, 119.1)
- added D52: 27V, Diodes_SMD:D_0603, F.Cu at (102.0, 119.1)
- added D53: 24.2V, Diodes_SMD:D_0603, F.Cu at (97.9, 119.1)
- added D54: 22.4V, Diodes_SMD:D_0603, F.Cu at (110.9, 119.1)
- added D55: LED, lib:LED_PLCC-2, F.Cu at (95.6, 113.5)
- added D56: LED, lib:LED_PLCC-2, F.Cu at (112.4, 113.5)
- added D57: LED, lib:LED_PLCC-2, F.Cu at (106.8, 113.5)
- added D58: LED, lib:LED_PLCC-2, F.Cu at (101.2, 113.5)
- added GND1: none, Measurement_Points:Test_Point_Keystone_5019_Minature, B.Cu at (186.5, 50.5)
- added GND2: none, Measurement_Points:Test_Point_Keystone_5019_Minature, B.Cu at (209.0, 88.0)
- added GND3: none, Measurement_Points:Test_Point_Keystone_5019_Minature, B.Cu at (130.0, 88.0)
- added GND4: none, Measurement_Points:Test_Point_Keystone_5019_Minature, B.Cu at (186.5, 106.0)
- added R13: 3k, Resistors_SMD:R_0603_HandSoldering, F.Cu at (93.4, 119.1)
- added VCC1: none, Measurement_Points:Test_Point_Keystone_5019_Minature, B.Cu at (157.5, 50.5)
- added VCC2: none, Measurement_Points:Test_Point_Keystone_5019_Minature, B.Cu at (209.0, 70.0)
- added VCC3: none, Measurement_Points:Test_Point_Keystone_5019_Minature, B.Cu at (130.0, 71.0)
- added VCC4: none, Measurement_Points:Test_Point_Keystone_5019_Minature, B.Cu at (157.0, 106.0)
- J5: value umbrella support -> umbrella hole
- J6: value BARREL_JACK -> PJ-002AH-SMT-TR; footprint Connectors:JACK_ALIM -> lib:PJ-002AH-SMT-TR
- moved J6 8.25 mm to (147.5, 53.5)
- moved F1 2.00 mm to (133.0, 59.5)
Connections:
- C1 pad 1: Vin -> Net-(C1-Pad1)
- F1 pad 1: Vin -> Net-(C1-Pad1)
- F1 pad 2: Net-(F1-Pad2) -> Vin
- J6 pad 1: Net-(F1-Pad2) -> Vin
- L1 pad 1: Vin -> Net-(C1-Pad1)
- SW1 pad 2: Net-(SW1-Pad2) -> Net-(C5-Pad1)
- SW1 pad 3: Net-(SW1-Pad3) -> Net-(R12-Pad2)
- U1 pad 3: Vin -> Net-(C1-Pad1)
- U1 pad 4: Vin -> Net-(C1-Pad1)
- U2 pad 14: Net-(U2-Pad14) -> Net-(C5-Pad1)
Other:
- board text added: "TEMP. 5600K"
- board text added: "focusaway.com v 1.15"
- board text removed: "focusaway.com"
